File: pcb_flat/front_back_view.kicad_pcb (KiCad board)
At the start: 2 copper layers, 119 x 40 mm, 8 parts, among them U1 nice!nano_v2, U1_back nice!nano_v2, U2 WeAct_BlackPill, U2_back WeAct_BlackPill, U3 DMC2038LVT_SOT-23-6, U3_back DMC2038LVT_SOT-23-6

Commit message: Stack battery on BlackPill (option B), update dimensions to 56 x 43 x 12.2
Co-Authored-By: Claude Opus 5.5 <noreply@anthropic.com>
Parts:
- added BT1: LiPo_30x25x5_on_BlackPill, pcb:LiPo_30x25x5_on_BlackPill, F.Cu at (150.0, 100.0)
- added BT1_back: LiPo_30x25x5_on_BlackPill, pcb:LiPo_30x25x5_on_BlackPill, B.Cu at (216.0, 100.0)
